Commit message: pantilt control

File: marr_gz/urdf/arms.xacro (robot description, xacro)
@@ -7,6 +7,8 @@
       <xacro:property name="arm_friction" value="0.01" />
       <xacro:property name="arm_damping" value="0.02" />
-      <xacro:property name="arm_lower_limit" value="${-5*pi/4}" />
-      <xacro:property name="arm_upper_limit" value="${pi/4}" />
+      <!--xacro:property name="arm_lower_limit" value="${-5*pi/4}" />
+      <xacro:property name="arm_upper_limit" value="${pi/4}" /-->
+      <xacro:property name="arm_lower_limit" value="${-2*pi}" />
+      <xacro:property name="arm_upper_limit" value="${2*pi}" />
       <xacro:property name="arm_max_effort" value="100" />
       <xacro:property name="arm_max_velocity" value="1.0" />
@@ -14,5 +16,5 @@
         <visual>
             <geometry>
-                <cylinder radius="${arm_radius}" length="${2*arm_radius+0.04}"/>
+                <cylinder radius="${arm_radius}" length="${2*arm_radius+0.08}"/>
             </geometry>
             <origin xyz="0.0 0.0 0.0" rpy="${pi/2} 0.0 0.0"/>
@@ -62,5 +64,5 @@
         <visual>
             <geometry>
-                <cylinder radius="${arm_radius}" length="${2*arm_radius+0.04}"/>
+                <cylinder radius="${arm_radius}" length="${2*arm_radius+0.08}"/>
             </geometry>
             <origin xyz="0.0 0.0 0.0" rpy="${pi/2} 0.0 0.0"/>
@@ -103,5 +105,5 @@
         <parent link="left_arm_body"/>
         <child link="left_arm"/>
-        <origin xyz="${arm_length/2} 0.02 0.0" rpy="0 0.0 0.0"/>
+        <origin xyz="${arm_length/2} 0.04 0.0" rpy="0 0.0 0.0"/>
       </joint>
       <!-- joint name="left_arm_tip_joint" type="fixed">
@@ -122,5 +124,5 @@
         <parent link="right_arm_body"/>
         <child link="right_arm"/>
-        <origin xyz="${arm_length/2} -0.02 0.0" rpy="0 0.0 0.0"/>
+        <origin xyz="${arm_length/2} -0.04 0.0" rpy="0 0.0 0.0"/>
       </joint>
   </xacro:macro>

File: marr_gz/urdf/pantilt.xacro (robot description, xacro)
@@ -3,6 +3,67 @@
   <xacro:macro name="pantilt" params="parent x y z">
     <link name="pantilt_base_link">
+        <visual>
+          <origin xyz="0 0 0.05" rpy="0 0 0" />
+          <geometry>
+            <cylinder radius="0.01" length="0.10"/>
+          </geometry>
+          <material name="black"/>
+        </visual>
+        <collision>
+          <origin xyz="0 0 0.05" rpy="0 0 0" />
+          <geometry>
+            <cylinder radius="0.01" length="0.10"/>
+          </geometry>
+        </collision>
+        <xacro:cylinder_inertial mass="0.10" radius="0.01" length="0.10"/>
+    </link>
+    <link name="pan_link">
+        <visual>
+            <geometry>
+                <cylinder radius="0.01" length="0.01"/>
+            </geometry>
+            <origin xyz="0.0 0.0 0.0" rpy="0.0 0.0 0.0"/>
+            <material name="blue"/>
+        </visual>
+        <collision>
+            <geometry>
+                <cylinder radius="0.01" length="0.01"/>
+            </geometry>
+            <origin xyz="0.0 0.0 0.0" rpy="0.0 0.0 0.0"/>
+        </collision>
+        <xacro:cylinder_inertial mass="0.05" radius="0.01" length="0.01"/>
+    </link>
+    <link name="tilt_link">
+        <visual>
+            <geometry>
+                <cylinder radius="0.01" length="0.014"/>
+            </geometry>
+            <origin xyz="0.0 0.0 0.0" rpy="${pi/2} 0.0 0.0"/>
+            <material name="green"/>
+        </visual>
+        <collision>
+            <geometry>
+                <cylinder radius="0.01" length="0.014"/>
+            </geometry>
+            <origin xyz="0.0 0.0 0.0" rpy="${pi/2} 0.0 0.0"/>
+        </collision>
+        <xacro:cylinder_inertial mass="0.05" radius="0.01" length="0.014"/>
     </link>
     <link name="pantilt_tip_link">
+        <visual>
+          <origin xyz="0 0 0" rpy="0 0 0" />
+          <geometry>
+            <cylinder radius="0.01" length="0.02"/>
+          </geometry>
+          <material name="black"/>
+        </visual>
+        <collision>
+          <origin xyz="0 0 0" rpy="0 0 0" />
+          <geometry>
+            <cylinder radius="0.01" length="0.02"/>
+          </geometry>
+          <material name="black"/>
+        </collision>
+        <xacro:cylinder_inertial mass="0.05" radius="0.01" length="0.02"/>
     </link>
     <joint name="pantilt_base_joint" type="fixed">
@@ -11,4 +72,27 @@
       <origin xyz="${x} ${y} ${z}" rpy="0.0 0.0 0.0"/>
     </joint>
+    <joint name="pantilt_pan_joint" type="revolute">
+      <parent link="pantilt_base_link"/>
+      <child link="pan_link"/>
+      <origin xyz="0 0 0.105" rpy="0.0 0.0 0.0"/>
+      <axis xyz="0.0 0.0 1.0"/>
+      <dynamics friction="0.01" damping="0.02" />
+      <limit lower="${-pi}" upper="${pi}"
+            effort="10" velocity="1.0"/>
+    </joint>
+    <joint name="pantilt_tilt_joint" type="revolute">
+      <parent link="pan_link"/>
+      <child link="tilt_link"/>
+      <origin xyz="0 0 0.015" rpy="0.0 0.0 0.0"/>
+      <axis xyz="0.0 1.0 0.0"/>
+      <dynamics friction="0.01" damping="0.02" />
+      <limit lower="${-pi/4}" upper="${pi/4}"
+            effort="10" velocity="1.0"/>
+    </joint>
+    <joint name="pantilt_tip_joint" type="fixed">
+      <parent link="tilt_link"/>
+      <child link="pantilt_tip_link"/>
+      <origin xyz="0.02 0 0.0" rpy="0.0 ${pi/2} 0.0"/>
+    </joint>
   </xacro:macro>
 </robot>

File: marr_gz/urdf/reacher.urdf.xacro (robot description, xacro)
@@ -1,4 +1,7 @@
 <?xml version="1.0"?>
 <robot name="reacher5" xmlns:xacro="http://ros.org/wiki/xacro">
+  <gazebo>
+      <self_collide>true</self_collide>
+  </gazebo>
   <xacro:arg name="namespace" default="" />
   <xacro:arg name="dof" default="2" />
@@ -9,5 +12,5 @@
   <xacro:include filename="$(find marr_gz)/urdf/inertia.xacro" />
   <xacro:include filename="$(find marr_gz)/urdf/sensors.xacro" />
-  <xacro:property name="base_mass" value="3.0" />
+  <xacro:property name="base_mass" value="5.0" />
   <xacro:property name="arm_radius" value="0.02" />
   <xacro:property name="arm_length" value="0.3" />
@@ -61,5 +64,5 @@
     <xacro:arm_joint_link_y name="arm_joint_link3" radius="${j_radius}" />
     <xacro:arm_joint_link_y name="arm_joint_link4" radius="${j_radius}" />
-    <xacro:arm_joint_link_x name="arm_joint_link5" radius="${j_radius}" />
+    <xacro:arm_joint_link_z name="arm_joint_link5" radius="${j_radius}" />
   </xacro:if>
   <xacro:if value="${$(arg dof) == 6}">
@@ -69,12 +72,12 @@
     <xacro:arm_joint_link_y name="arm_joint_link4" radius="${j_radius}" />
     <xacro:arm_joint_link_y name="arm_joint_link5" radius="${j_radius}" />
-    <xacro:arm_joint_link_x name="arm_joint_link6" radius="${j_radius}" />
+    <xacro:arm_joint_link_z name="arm_joint_link6" radius="${j_radius}" />
   </xacro:if>
   <xacro:tip_link name="tip_link" />
   <!-- Joints -->
-  <xacro:fixed_joint name="base_joint" parent="base_footprint" child="base_link" x="0" z="0" />
+  <xacro:fixed_joint name="base_joint" parent="base_link" child="base_footprint" x="0" z="-0.05" />
   <xacro:if value="${$(arg dof) == 2}">
     <xacro:revolute_joint_z name="arm_joint1" parent="base_link" child="arm_joint_link1"
-     x="0" z="0.1" lower="${-pi}" upper="${pi}" />
+     x="0" z="${0.1+0.025}" lower="${-pi}" upper="${pi}" />
    <xacro:revolute_joint_z name="arm_joint2" parent="arm_link1" child="arm_joint_link2"
      x="${arm_length/2}" z="0" lower="${-7/8*pi}" upper="${7/8*pi}" />
@@ -85,5 +88,5 @@
   <xacro:if value="${$(arg dof) == 3}">
     <xacro:revolute_joint_z name="arm_joint1" parent="base_link" child="arm_joint_link1"
-     x="0" z="0.1" lower="${-pi}" upper="${pi}" />
+     x="0" z="${0.1+0.025}" lower="${-pi}" upper="${pi}" />
     <xacro:revolute_joint_z name="arm_joint2" parent="arm_link1" child="arm_joint_link2"
      x="${arm_length/2}" z="0" lower="${-1.8}" upper="${1.8}" />
@@ -97,10 +100,10 @@
   <xacro:if value="${$(arg dof) == 4}">
     <xacro:revolute_joint_z name="arm_joint1" parent="base_link" child="arm_joint_link1"
-     x="0" z="0.1" lower="${-pi}" upper="${pi}" />
+     x="0" z="${0.1+0.025}" lower="${-pi}" upper="${pi}" />
     <xacro:revolute_joint_y name="arm_joint2" parent="arm_link1" child="arm_joint_link2"
      x="0" z="0.05" lower="${-1.8}" upper="${1.8}" />
     <xacro:revolute_joint_y name="arm_joint3" parent="arm_link2" child="arm_joint_link3"
      x="${arm_length/2}" z="0" lower="${-1.8}" upper="${1.8}" />
-    <xacro:revolute_joint_x name="arm_joint4" parent="arm_link3" child="arm_joint_link4"
+    <xacro:revolute_joint_y name="arm_joint4" parent="arm_link3" child="arm_joint_link4"
      x="${arm_length/2}" z="0" lower="${-1.8}" upper="${1.8}" />
     <xacro:fixed_joint name="arm_joint1b" parent="arm_joint_link1" child="arm_link1" x="0" z="0.05" />
@@ -112,5 +115,5 @@
   <xacro:if value="${$(arg dof) == 5}">
     <xacro:revolute_joint_z name="arm_joint1" parent="base_link" child="arm_joint_link1"
-     x="0" z="0.1" lower="${-pi}" upper="${pi}" />
+     x="0" z="${0.1+0.025}" lower="${-pi}" upper="${pi}" />
     <xacro:revolute_joint_y name="arm_joint2" parent="arm_link1" child="arm_joint_link2"
      x="0" z="0.05" lower="${-1.8}" upper="${1.8}" />
@@ -119,5 +122,5 @@
     <xacro:revolute_joint_y name="arm_joint4" parent="arm_link3" child="arm_joint_link4"
      x="${arm_length/2}" z="0" lower="${-1.8}" upper="${1.8}" />
-    <xacro:revolute_joint_x name="arm_joint5" parent="arm_link4" child="arm_joint_link5"
+    <xacro:revolute_joint_z name="arm_joint5" parent="arm_link4" child="arm_joint_link5"
      x="${arm_length/2}" z="0" lower="${-1.8}" upper="${1.8}" />
     <xacro:fixed_joint name="arm_joint1b" parent="arm_joint_link1" child="arm_link1" x="0" z="0.05" />
@@ -130,5 +133,5 @@
   <xacro:if value="${$(arg dof) == 6}">
     <xacro:revolute_joint_z name="arm_joint1" parent="base_link" child="arm_joint_link1"
-     x="0" z="0.1" lower="${-pi}" upper="${pi}" />
+     x="0" z="${0.1+0.025}" lower="${-pi}" upper="${pi}" />
     <xacro:revolute_joint_y name="arm_joint2" parent="arm_link1" child="arm_joint_link2"
      x="0" z="0.05" lower="${-1.8}" upper="${1.8}" />
@@ -139,5 +142,5 @@
     <xacro:revolute_joint_y name="arm_joint5" parent="arm_link4" child="arm_joint_link5"
      x="${arm_length/2}" z="0" lower="${-1.8}" upper="${1.8}" />
-    <xacro:revolute_joint_x name="arm_joint6" parent="arm_link5" child="arm_joint_link6"
+    <xacro:revolute_joint_z name="arm_joint6" parent="arm_link5" child="arm_joint_link6"
      x="${arm_length/2}" z="0" lower="${-1.8}" upper="${1.8}" />
     <xacro:fixed_joint name="arm_joint1b" parent="arm_joint_link1" child="arm_link1" x="0" z="0.05" />

File: marr_gz/urdf/reacher_base.urdf.xacro (robot description, xacro)
@@ -104,12 +104,5 @@
         <visual>
             <geometry>
-                <cylinder radius="0.1" length="0.05"/>
-            </geometry>
-            <origin xyz="0.0 0.0 0.0" rpy="0.0 0.0 0.0"/>
-            <material name="black"/>
-        </visual>
-        <visual>
-            <geometry>
-                <cylinder radius="0.05" length="0.05"/>
+                <cylinder radius="0.2" length="0.1"/>
             </geometry>
             <origin xyz="0.0 0.0 0.05" rpy="0.0 0.0 0.0"/>
@@ -118,9 +111,9 @@
         <collision>
             <geometry>
-                <cylinder radius="0.1" length="0.1"/>
+                <cylinder radius="0.2" length="0.1"/>
             </geometry>
-            <origin xyz="0.0 0.0 0.0" rpy="0.0 0.0 0.0"/>
+            <origin xyz="0.0 0.0 0.05" rpy="0.0 0.0 0.0"/>
         </collision>
-        <xacro:cylinder_inertial mass="${base_mass}" radius="0.1" length="0.1" />
+        <xacro:cylinder_inertial mass="${base_mass}" radius="0.2" length="0.1" />
       </link>
   </xacro:macro>

File: marr_gz/urdf/sensors.xacro (robot description, xacro)
@@ -79,4 +79,31 @@
     </xacro:macro>
     <xacro:macro name="rgb" params="parent x y z">
+      <link name="camera_link">
+        <visual>
+          <origin xyz="0 0 0.05" rpy="0 0 0" />
+          <geometry>
+            <cylinder radius="0.01" length="0.10"/>
+          </geometry>
+          <material name="black"/>
+        </visual>
+        <visual>
+          <origin xyz="0.01 0 ${0.10+0.02}" rpy="0 ${pi/2+0.6} 0" />
+          <geometry>
+            <cylinder radius="0.02" length="0.02"/>
+          </geometry>
+          <material name="black"/>
+        </visual>
+      </link>
+      <link name="camera_optical_link" />
+      <joint name="camera_joint" type="fixed">
+        <parent link="${parent}"/>
+        <child link="camera_link"/>
+        <origin xyz="0 0.0 0.15" rpy="0.0 0.0 0.0"/>
+      </joint>
+      <joint name="camera_optical_joint" type="fixed">
+        <parent link="camera_link"/>
+        <child link="camera_optical_link"/>
+        <origin xyz="0.02 0 ${0.10+0.02}" rpy="0 0.6 0"/>
+      </joint>
     </xacro:macro>
     <xacro:macro name="rgbd" params="parent x y z">

File: marr_gz/urdf/wheeled.urdf.xacro (robot description, xacro)
@@ -151,5 +151,5 @@
   </xacro:if>
   <xacro:if value="$(arg use_pantilt)">
-    <xacro:pantilt parent="base_link" x="0.1" y="0.0" z="0.152" />
+    <xacro:pantilt parent="base_link" x="0.0" y="0.0" z="0.152" />
   </xacro:if>
   <!-- sensors -->
@@ -230,4 +230,36 @@
     </xacro:if>
     <xacro:if value="$(arg use_pantilt)">
+    <joint name="pantilt_pan_joint">
+      <command_interface name="effort">
+        <param name="min">-10</param>
+        <param name="max">10</param>
+      </command_interface>
+      <command_interface name="velocity">
+        <param name="min">-1</param>
+        <param name="max">1</param>
+      </command_interface>
+      <command_interface name="position">
+        <param name="min">-100</param>
+        <param name="max">100</param>
+      </command_interface>
+      <state_interface name="position"/>
+      <state_interface name="velocity"/>
+    </joint>
+    <joint name="pantilt_tilt_joint">
+      <command_interface name="effort">
+        <param name="min">-10</param>
+        <param name="max">10</param>
+      </command_interface>
+      <command_interface name="velocity">
+        <param name="min">-1</param>
+        <param name="max">1</param>
+      </command_interface>
+      <command_interface name="position">
+        <param name="min">-100</param>
+        <param name="max">100</param>
+      </command_interface>
+      <state_interface name="position"/>
+      <state_interface name="velocity"/>
+    </joint>
     </xacro:if>
   </ros2_control>
