Commit message: wheeled sensors

File: marr_gz/urdf/pantilt.xacro (robot description, xacro)
@@ -96,3 +96,90 @@
     </joint>
   </xacro:macro>
+  <xacro:macro name="camera_base" params="parent x y z">
+    <link name="pantilt_base_link">
+        <visual>
+          <origin xyz="0 0 0.05" rpy="0 0 0" />
+          <geometry>
+            <cylinder radius="0.01" length="0.10"/>
+          </geometry>
+          <material name="black"/>
+        </visual>
+        <collision>
+          <origin xyz="0 0 0.05" rpy="0 0 0" />
+          <geometry>
+            <cylinder radius="0.01" length="0.10"/>
+          </geometry>
+        </collision>
+        <xacro:cylinder_inertial mass="0.10" radius="0.01" length="0.10"/>
+    </link>
+    <link name="pan_link">
+        <visual>
+            <geometry>
+                <cylinder radius="0.01" length="0.01"/>
+            </geometry>
+            <origin xyz="0.0 0.0 0.0" rpy="0.0 0.0 0.0"/>
+            <material name="black"/>
+        </visual>
+        <collision>
+            <geometry>
+                <cylinder radius="0.01" length="0.01"/>
+            </geometry>
+            <origin xyz="0.0 0.0 0.0" rpy="0.0 0.0 0.0"/>
+        </collision>
+        <xacro:cylinder_inertial mass="0.05" radius="0.01" length="0.01"/>
+    </link>
+    <link name="tilt_link">
+        <visual>
+            <geometry>
+                <cylinder radius="0.01" length="0.014"/>
+            </geometry>
+            <origin xyz="0.0 0.0 0.0" rpy="${pi/2} 0.0 0.0"/>
+            <material name="black"/>
+        </visual>
+        <collision>
+            <geometry>
+                <cylinder radius="0.01" length="0.014"/>
+            </geometry>
+            <origin xyz="0.0 0.0 0.0" rpy="${pi/2} 0.0 0.0"/>
+        </collision>
+        <xacro:cylinder_inertial mass="0.05" radius="0.01" length="0.014"/>
+    </link>
+    <link name="pantilt_tip_link">
+        <visual>
+          <origin xyz="0 0 0" rpy="0 0 0" />
+          <geometry>
+            <cylinder radius="0.01" length="0.02"/>
+          </geometry>
+          <material name="black"/>
+        </visual>
+        <collision>
+          <origin xyz="0 0 0" rpy="0 0 0" />
+          <geometry>
+            <cylinder radius="0.01" length="0.02"/>
+          </geometry>
+          <material name="black"/>
+        </collision>
+        <xacro:cylinder_inertial mass="0.05" radius="0.01" length="0.02"/>
+    </link>
+    <joint name="pantilt_base_joint" type="fixed">
+      <parent link="${parent}"/>
+      <child link="pantilt_base_link"/>
+      <origin xyz="${x} ${y} ${z}" rpy="0.0 0.0 0.0"/>
+    </joint>
+    <joint name="pantilt_pan_joint" type="fixed">
+      <parent link="pantilt_base_link"/>
+      <child link="pan_link"/>
+      <origin xyz="0 0 0.105" rpy="0.0 0.0 0.0"/>
+    </joint>
+    <joint name="pantilt_tilt_joint" type="fixed">
+      <parent link="pan_link"/>
+      <child link="tilt_link"/>
+      <origin xyz="0 0 0.015" rpy="0.0 0.0 0.0"/>
+    </joint>
+    <joint name="pantilt_tip_joint" type="fixed">
+      <parent link="tilt_link"/>
+      <child link="pantilt_tip_link"/>
+      <origin xyz="0.02 0 0.0" rpy="0.0 ${pi/2} 0.0"/>
+    </joint>
+  </xacro:macro>
 </robot>

File: marr_gz/urdf/sensors.xacro (robot description, xacro)
@@ -81,16 +81,9 @@
       <link name="camera_link">
         <visual>
-          <origin xyz="0 0 0.05" rpy="0 0 0" />
           <geometry>
-            <cylinder radius="0.01" length="0.10"/>
+            <cylinder radius="0.005" length="0.006"/>
           </geometry>
-          <material name="black"/>
-        </visual>
-        <visual>
-          <origin xyz="0.01 0 ${0.10+0.02}" rpy="0 ${pi/2+0.6} 0" />
-          <geometry>
-            <cylinder radius="0.02" length="0.02"/>
-          </geometry>
-          <material name="black"/>
+          <material name="grey"/>
+          <origin xyz="0 0 0" rpy="0 0 0" />
         </visual>
       </link>
@@ -99,13 +92,69 @@
         <parent link="${parent}"/>
         <child link="camera_link"/>
-        <origin xyz="0 0.0 0.15" rpy="0.0 0.0 0.0"/>
+        <origin xyz="0 0 0.013" rpy="0.0 0.0 0.0"/>
       </joint>
       <joint name="camera_optical_joint" type="fixed">
         <parent link="camera_link"/>
         <child link="camera_optical_link"/>
-        <origin xyz="0.02 0 ${0.10+0.02}" rpy="0 0.6 0"/>
+        <origin xyz="0.006 0 0" rpy="0 ${-pi/2} 0"/>
+      </joint>
+      <gazebo reference="camera_optical_link">
+        <sensor name="camera" type="camera">
+          <camera>
+            <horizontal_fov>2.0</horizontal_fov>
+            <image>
+              <width>640</width>
+              <height>480</height>
+              <format>R8G8B8</format>
+            </image>
+            <clip>
+              <near>0.001</near>
+              <far>15</far>
+            </clip>
+            <noise>
+              <type>gaussian</type>
+              <!-- Noise is sampled independently per pixel on each frame.
+                   That pixel's noise value is added to each of its color
+                   channels, which at that point lie in the range [0,1]. -->
+              <mean>0.0</mean>
+              <stddev>0.007</stddev>
+            </noise>
+            <camera_info_topic>camera/camera_info</camera_info_topic>
+          </camera>
+          <always_on>1</always_on>
+          <update_rate>10</update_rate>
+          <visualize>true</visualize>
+          <topic>camera/image</topic>
+        </sensor>
+      </gazebo>
+    </xacro:macro>
+    <xacro:macro name="rgbd" params="parent x y z">
+      <link name="camera_link">
+        <visual>
+          <geometry>
+            <cylinder radius="0.005" length="0.006"/>
+          </geometry>
+          <material name="grey"/>
+          <origin xyz="0 -0.006 0" rpy="0 0 0" />
+        </visual>
+        <visual>
+          <geometry>
+            <cylinder radius="0.005" length="0.006"/>
+          </geometry>
+          <material name="grey"/>
+          <origin xyz="0 0.006 0" rpy="0 0 0" />
+        </visual>
+      </link>
+      <link name="camera_optical_link" />
+      <joint name="camera_joint" type="fixed">
+        <parent link="${parent}"/>
+        <child link="camera_link"/>
+        <origin xyz="0 0 0.013" rpy="0.0 0.0 0.0"/>
+      </joint>
+      <joint name="camera_optical_joint" type="fixed">
+        <parent link="camera_link"/>
+        <child link="camera_optical_link"/>
+        <origin xyz="0.006 0 0" rpy="0 0.0 0"/>
       </joint>
     </xacro:macro>
-    <xacro:macro name="rgbd" params="parent x y z">
-    </xacro:macro>
 </robot>

File: marr_gz/urdf/wheeled.urdf.xacro (robot description, xacro)
@@ -167,5 +167,6 @@
   </xacro:if>
   <xacro:if value="${u_rgb and not u_pantilt}">
-    <xacro:rgb parent="base_link" x="0.1" y="0.0" z="0.5" />
+    <xacro:camera_base parent="base_link" x="0.0" y="0.0" z="0.152" />
+    <xacro:rgb parent="pantilt_tip_link" x="0.1" y="0.0" z="0.5" />
   </xacro:if>
   <xacro:if value="${u_rgbd and u_pantilt}">
@@ -173,5 +174,6 @@
   </xacro:if>
   <xacro:if value="${u_rgbd and not u_pantilt}">
-    <xacro:rgbd parent="base_link" x="0.1" y="0.0" z="0.5" />
+    <xacro:camera_base parent="base_link" x="0.0" y="0.0" z="0.152" />
+    <xacro:rgbd parent="pantilt_tip_link" x="0.1" y="0.0" z="0.5" />
   </xacro:if>
   <ros2_control name="GazeboSimSystem" type="system">
