Commit message: rgbd and odom fine tuning

File: marr_gz/urdf/sensors.xacro (robot description, xacro)
@@ -97,5 +97,5 @@
         <parent link="camera_link"/>
         <child link="camera_optical_link"/>
-        <origin xyz="0.006 0 0" rpy="0 ${-pi/2} 0"/>
+        <origin xyz="0 0 0.006" rpy="0 ${-pi/2} 0"/>
       </joint>
       <gazebo reference="camera_optical_link">
@@ -143,5 +143,5 @@
           </geometry>
           <material name="grey"/>
-          <origin xyz="0 0.006 0" rpy="0 0 0" />
+          <origin xyz="0 0 0.006" rpy="0 0 0" />
         </visual>
       </link>
@@ -155,6 +155,51 @@
         <parent link="camera_link"/>
         <child link="camera_optical_link"/>
-        <origin xyz="0.006 0 0" rpy="0 0.0 0"/>
-      </joint>
+        <origin xyz="0 0 0.006" rpy="0 ${-pi/2} 0"/>
+      </joint>
+      <gazebo reference="camera_optical_link">
+        <sensor name="camera" type="rgbd_camera">
+          <camera>
+            <horizontal_fov>2.0</horizontal_fov>
+            <image>
+              <width>640</width>
+              <height>480</height>
+              <format>R8G8B8</format>
+            </image>
+            <clip>
+              <near>0.001</near>
+              <far>15</far>
+            </clip>
+            <noise>
+              <type>gaussian</type>
+              <!-- Noise is sampled independently per pixel on each frame.
+                   That pixel's noise value is added to each of its color
+                   channels, which at that point lie in the range [0,1]. -->
+              <mean>0.0</mean>
+              <stddev>0.007</stddev>
+            </noise>
+            <!-- camera_info_topic>camera/camera_info</camera_info_topic -->
+          </camera>
+          <depth_camera>
+            <image>
+              <width>640</width>
+              <height>480</height>
+              <format>R_FLOAT32</format>
+              <!-- format>16UC1</format -->
+            </image>
+            <clip>
+              <near>0.1</near>
+              <far>10</far>
+            </clip>
+            <point_cloud>
+                <format>xyz</format>
+            </point_cloud>
+          </depth_camera>
+          <always_on>1</always_on>
+          <update_rate>10</update_rate>
+          <visualize>true</visualize>
+          <topic>camera</topic>
+          <gz_frame_id>camera_optical_link</gz_frame_id>  <!-- ignore warning not defined in SDF -->
+        </sensor>
+      </gazebo>
     </xacro:macro>
 </robot>

File: marr_gz/urdf/wheeled.urdf.xacro (robot description, xacro)
@@ -40,4 +40,21 @@
     <xacro:box_inertial mass="0.2" x_dim="0.5" y_dim="0.4" z_dim="0.3"/>
   </link>
+  <!-- to balance weight on the bottom and between the wheels -->
+  <link name="battery_link">
+    <visual>
+        <geometry>
+            <box size="0.1 0.2 0.1"/>
+        </geometry>
+        <origin xyz="0.0 0.0 0.0" rpy="0.0 0.0 0.0"/>
+        <material name="black"/>
+    </visual>
+    <collision>
+        <geometry>
+            <box size="0.1 0.2 0.1"/>
+        </geometry>
+        <origin xyz="0.0 0.0 0.0" rpy="0.0 0.0 0.0"/>
+    </collision>
+    <xacro:box_inertial mass="0.5" x_dim="0.1" y_dim="0.2" z_dim="0.1"/>
+  </link>
   <link name="left_wheel">
     <visual>
@@ -124,5 +141,10 @@
     <parent link="base_footprint"/>
     <child link="base_link"/>
-    <origin xyz="0.0 0.0 0.50" rpy="0.0 0.0 0.0"/>
+    <origin xyz="-0.1 0.0 0.15" rpy="0.0 0.0 0.0"/>
+  </joint>
+  <joint name="battery_joint" type="fixed">
+    <parent link="base_link"/>
+    <child link="battery_link"/>
+    <origin xyz="0.1 0.0 -0.08" rpy="0.0 0.0 0.0"/>
   </joint>
   <joint name="left_wheel_joint" type="continuous">
@@ -132,5 +154,5 @@
     <axis xyz="0.0 1.0 0.0"/>
     <dynamics damping="0.2" friction="1.0"/>
-    <limit effort="100" velocity="1.0"/>
+    <limit effort="100" velocity="10.0"/>
   </joint>
   <joint name="right_wheel_joint" type="continuous">
@@ -140,5 +162,5 @@
     <axis xyz="0.0 1.0 0.0"/>
     <dynamics damping="0.2" friction="1.0"/>
-    <limit effort="100" velocity="1.0"/>
+    <limit effort="100" velocity="10.0"/>
   </joint>
   <joint name="caster_wheel_joint" type="fixed">
@@ -273,4 +295,14 @@
       </ros>
       <parameters>$(find marr_gz)/config/wheeled_controllers.yaml</parameters>
+    </plugin>
+  </gazebo>
+  <gazebo>
+    <!-- Ground truth publisher -->
+    <plugin
+        filename="gz-sim-pose-publisher-system"
+        name="gz::sim::systems::PosePublisher">
+        <use_pose_vector_msg>false</use_pose_vector_msg>
+        <publish_model_pose>true</publish_model_pose>
+        <publish_nested_model_pose>true</publish_nested_model_pose>
     </plugin>
   </gazebo>
