Commit message: reacher sensors

File: marr_gz/urdf/reacher.urdf.xacro (robot description, xacro)
@@ -154,14 +154,14 @@
   <!-- sensors -->
   <xacro:if value="$(arg use_imu)">
-    <xacro:imu parent="tip_link" x="-0.1" y="0.0" z="0.152" />
+    <xacro:imu parent="tip_link" x="0.0" y="0.0" z="-0.06" />
   </xacro:if>
   <xacro:if value="$(arg use_lidar)">
-    <xacro:lidar parent="tip_link" x="0.1" y="0.0" z="0.155" />
+    <xacro:lidar parent="tip_link" x="0.0" y="0.0" z="0.075" />
   </xacro:if>
   <xacro:if value="$(arg use_rgb)">
-    <xacro:rgb parent="tip_link" x="0.1" y="0.0" z="0.5" />
+    <xacro:rgb parent="tip_link" x="0.05" y="0.0" z="0" p="${pi/2}" />
   </xacro:if>
   <xacro:if value="$(arg use_rgbd)">
-    <xacro:rgbd parent="tip_link" x="0.1" y="0.0" z="0.5" />
+    <xacro:rgbd parent="tip_link" x="0.05" y="0.0" z="0" p="${pi/2}" />
   </xacro:if>
   <ros2_control name="GazeboSimSystem" type="system">

File: marr_gz/urdf/sensors.xacro (robot description, xacro)
@@ -78,5 +78,5 @@
       </gazebo>
     </xacro:macro>
-    <xacro:macro name="rgb" params="parent x y z">
+    <xacro:macro name="rgb" params="parent x y z p">
       <link name="camera_link">
         <visual>
@@ -92,5 +92,5 @@
         <parent link="${parent}"/>
         <child link="camera_link"/>
-        <origin xyz="0 0 0.013" rpy="0.0 0.0 0.0"/>
+        <origin xyz="${x} ${y} ${z}" rpy="0.0 ${p} 0.0"/>
       </joint>
       <joint name="camera_optical_joint" type="fixed">
@@ -129,5 +129,5 @@
       </gazebo>
     </xacro:macro>
-    <xacro:macro name="rgbd" params="parent x y z">
+    <xacro:macro name="rgbd" params="parent x y z p">
       <link name="camera_link">
         <visual>
@@ -143,5 +143,5 @@
           </geometry>
           <material name="grey"/>
-          <origin xyz="0 0 0.006" rpy="0 0 0" />
+          <origin xyz="0 0.006 0" rpy="0 0 0" />
         </visual>
       </link>
@@ -150,5 +150,5 @@
         <parent link="${parent}"/>
         <child link="camera_link"/>
-        <origin xyz="0 0 0.013" rpy="0.0 0.0 0.0"/>
+        <origin xyz="${x} ${y} ${z}" rpy="0.0 ${p} 0.0"/>
       </joint>
       <joint name="camera_optical_joint" type="fixed">

File: marr_gz/urdf/wheeled.urdf.xacro (robot description, xacro)
@@ -186,16 +186,16 @@
   <xacro:property name="u_pantilt" value="$(arg use_pantilt)"/>
   <xacro:if value="${u_rgb and u_pantilt}">
-    <xacro:rgb parent="pantilt_tip_link" x="0.1" y="0.0" z="0.5" />
+    <xacro:rgb parent="pantilt_tip_link" x="0.0" y="0.0" z="0.013" p="0" />
   </xacro:if>
   <xacro:if value="${u_rgb and not u_pantilt}">
     <xacro:camera_base parent="base_link" x="0.0" y="0.0" z="0.152" />
-    <xacro:rgb parent="pantilt_tip_link" x="0.1" y="0.0" z="0.5" />
+    <xacro:rgb parent="pantilt_tip_link" x="0.0" y="0.0" z="0.013" p="0" />
   </xacro:if>
   <xacro:if value="${u_rgbd and u_pantilt}">
-    <xacro:rgbd parent="pantilt_tip_link" x="0.1" y="0.0" z="0.5" />
+    <xacro:rgbd parent="pantilt_tip_link" x="0.0" y="0.0" z="0.013" p="0" />
   </xacro:if>
   <xacro:if value="${u_rgbd and not u_pantilt}">
     <xacro:camera_base parent="base_link" x="0.0" y="0.0" z="0.152" />
-    <xacro:rgbd parent="pantilt_tip_link" x="0.1" y="0.0" z="0.5" />
+    <xacro:rgbd parent="pantilt_tip_link" x="0.0" y="0.0" z="0.013" p="0" />
   </xacro:if>
   <ros2_control name="GazeboSimSystem" type="system">
